Commit message: added dae file

File: cuarm.urdf (robot description, URDF)
Before this commit: robot cuarm, 12 links, 11 joints
Links:
- added link gripper_dummy_link; collision cylinder length=0.0 radius=0.03; visual cylinder length=0.0 radius=0.03
- added link gripper_tip; collision cylinder length=0.05 radius=0.02; visual cylinder length=0.05 radius=0.02
Joints:
- added joint dummy_joint: type revolute, parent gripper_hand, child gripper_dummy_link, origin xyz=0 0 0.17 rpy=0 0 0, axis 1 0 0, limit lower=-1.57 upper=1.57 effort=1.0 velocity=0.3
- added joint fixed_link_to_tip: type fixed, parent gripper_dummy_link, child gripper_tip, origin xyz=0 0 0 rpy=0 0 0

File: cuarm.xacro (robot description, xacro)
@@ -226,3 +226,21 @@
         <xacro:color_blue />
     </xacro:cyl>
+    <joint name="dummy_joint" type="revolute">
+        <origin xyz="0 0 0.17" rpy="0 0 0" />
+        <axis xyz="1 0 0" />
+        <parent link="gripper_hand" />
+        <child link="gripper_dummy_link" />
+        <limit lower="-1.57" upper="1.57" velocity="0.3" effort="1.0" />
+    </joint>
+    <xacro:cyl name="gripper_dummy_link" radius="0.03" length="0.0">
+        <xacro:color_magenta />
+    </xacro:cyl>
+    <joint name="fixed_link_to_tip" type="fixed">
+        <origin xyz="0 0 0" rpy="0 0 0" />
+        <parent link="gripper_dummy_link" />
+        <child link="gripper_tip" />
+    </joint>
+    <xacro:cyl name="gripper_tip" radius="0.02" length="0.05">
+        <xacro:color_magenta />
+    </xacro:cyl>
 </robot>
